Commit message: Collision and approx limits for moveit

File: urdf/xArm.urdf (robot description, URDF)
Before this commit: robot xArm, 7 links, 6 joints
Links:
- link link1: geometry collision box size=0.044 0.0285 0.0065; collision box size=0.044 0.0285 0.023
- link link2: geometry collision box size=0.025 0.002 0.045; collision box size=0.025 0.002 0.045
- link link3: geometry collision box size=0.023 0.0285 0.004; collision box size=0.023 0.0285 0.004
- link link4: geometry collision box size=0.025 0.002 0.064; collision box size=0.025 0.002 0.064
- link link5: geometry collision cylinder length=0.004 radius=0.01; visual cylinder length=0.004 radius=0.01
Joints:
- joint arm1: limit (none) -> lower=-3.0 upper=3.0 effort=10.0 velocity=0.5; type continuous -> revolute
- joint arm2: limit (none) -> lower=-3.0 upper=3.0 effort=10.0 velocity=0.5; type continuous -> revolute
- joint arm3: limit (none) -> lower=-3.0 upper=3.0 effort=10.0 velocity=0.5; type continuous -> revolute
- joint arm4: limit (none) -> lower=-3.0 upper=3.0 effort=10.0 velocity=0.5; type continuous -> revolute
- joint arm5: limit (none) -> lower=-3.0 upper=3.0 effort=10.0 velocity=0.5; type continuous -> revolute
